File: CAD/USB_Connections.kicad_sch (KiCad schematic)
At the start: 7 parts, among them J8 USB_C_Plug_USB2.0

Commit message: Layout progress
Connections:
- net D+: now also D19.2 (K); no longer D19.1 (K)
- net D-: now also D19.1 (K); no longer D19.2 (K)
Changed lines of the file:
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@@
 (kicad_sch (version 20230121) (generator eeschema)
   (paper "A4")
-  (junction (at 114.3 91.44) (diameter 0) (color 0 0 0 0)
+  (junction (at 119.38 91.44) (diameter 0) (color 0 0 0 0)
   )
   (junction (at 74.93 123.19) (diameter 0) (color 0 0 0 0)
   )
+  (junction (at 114.3 86.36) (diameter 0) (color 0 0 0 0)
+  )
   (junction (at 67.31 114.3) (diameter 0) (color 0 0 0 0)
-  )
-  (junction (at 119.38 86.36) (diameter 0) (color 0 0 0 0)
   )
   (junction (at 67.31 123.19) (diameter 0) (color 0 0 0 0)
@@
     (stroke (width 0) (type default))
   )
-  (wire (pts (xy 90.17 91.44) (xy 114.3 91.44))
+  (wire (pts (xy 90.17 91.44) (xy 119.38 91.44))
     (stroke (width 0) (type default))
   )
-  (wire (pts (xy 90.17 86.36) (xy 119.38 86.36))
+  (wire (pts (xy 90.17 86.36) (xy 114.3 86.36))
     (stroke (width 0) (type default))
   )
@@
   )
   (wire (pts (xy 67.31 123.19) (xy 74.93 123.19))
-    (stroke (width 0) (type default))
-  )
-  (wire (pts (xy 119.38 86.36) (xy 127 86.36))
     (stroke (width 0) (type default))
   )
@@
     (stroke (width 0) (type default))
   )
+  (wire (pts (xy 119.38 91.44) (xy 119.38 93.98))
+    (stroke (width 0) (type default))
+  )
+  (wire (pts (xy 119.38 91.44) (xy 127 91.44))
+    (stroke (width 0) (type default))
+  )
   (wire (pts (xy 58.42 123.19) (xy 67.31 123.19))
     (stroke (width 0) (type default))
@@
   )
   (wire (pts (xy 58.42 115.57) (xy 58.42 114.3))
-    (stroke (width 0) (type default))
-  )
-  (wire (pts (xy 119.38 86.36) (xy 119.38 93.98))
-    (stroke (width 0) (type default))
-  )
-  (wire (pts (xy 114.3 91.44) (xy 127 91.44))
     (stroke (width 0) (type default))
   )
@@
     (stroke (width 0) (type default))
   )
-  (wire (pts (xy 114.3 91.44) (xy 114.3 93.98))
+  (wire (pts (xy 90.17 73.66) (xy 91.44 73.66))
     (stroke (width 0) (type default))
   )
-  (wire (pts (xy 90.17 73.66) (xy 91.44 73.66))
+  (wire (pts (xy 114.3 86.36) (xy 127 86.36))
     (stroke (width 0) (type default))
   )
@@
     (stroke (width 0) (type default))
   )
+  (wire (pts (xy 114.3 93.98) (xy 114.3 86.36))
+    (stroke (width 0) (type default))
+  )
