File: CAD/USB_Connections.kicad_sch (KiCad schematic)
At the start: 7 parts, among them J8 USB_C_Plug_USB2.0

Commit message: updates
Parts:
- C8: symbol Device:C_Small -> BadgePirates:C_.1uf_0805; MFG (none) -> TORCH; MFG_PN (none) -> CT41G-0805-2X1-50V-0.1μF-K(N); Vendor1 (none) -> LCSC; Vendor1_PN (none) -> C126469; Vendor1_URL (none) -> https://www.lcsc.com/product-detail/Multilayer-Ceramic-Capa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
- D19: MFG (none) -> TECH PUBLIC; MFG_PN (none) -> PESD2USB3UV-TR; Vendor1 (none) -> LCSC; Vendor1_URL (none) -> https://www.lcsc.com/product-detail/span-style-background-c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; Vendor_PN (none) -> C7202955
- J8: MFG (none) -> Jing Extension of the Electronic Co.; MFG_PN (none) -> 918-418K2023S40019; Vendor1 (none) -> LCSC; Vendor1_PN (none) -> C709035; Vendor1_URL (none) -> https://www.lcsc.com/product-detail/USB-Connectors_Jing-Ext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
- R10: symbol Device:R_Small_US -> BadgePirates:R_5.1k_1206; MFG (none) -> YEGEO; MFG_PN (none) -> RC1206FR-075K1L; Vendor1 (none) -> LCSC; Vendor1_PN (none) -> C163372; Vendor1_URL (none) -> https://www.lcsc.com/product-detail/Chip-Resistor-Surface-M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
- R11: MFG (none) -> YEGEO; MFG_PN (none) -> RC1206FR-075K1L; Vendor1 (none) -> LCSC; Vendor1_PN (none) -> C163372; Vendor1_URL (none) -> https://www.lcsc.com/product-detail/Chip-Resistor-Surface-M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
- R7: MFG (none) -> YAGEO; MFG_PN (none) -> RC1206FR-071ML; Vendor1 (none) -> LCSC; Vendor1_PN (none) -> C108083; Vendor1_URL (none) -> https://www.lcsc.com/product-detail/Chip-Resistor-Surface-M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
- R8: MFG (none) -> UNI-ROYAL(Uniroyal Elec); MFG_PN (none) -> 1206W4F0000T5E; Vendor1 (none) -> LCSC; Vendor1_PN (none) -> C17888; Vendor1_URL (none) -> https://www.lcsc.com/product-detail/Chip-Resistor-Surface-M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
Changed lines of the file:
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@@
       (effects (font (size 1.27 1.27)) hide)
     )
-    (property "Datasheet" "~" (at 67.31 118.11 0)
+    (property "Datasheet" "https://datasheet.lcsc.com/lcsc/2304140030_YAGEO-RC1206FR-071ML_C108083.pdf" (at 67.31 118.11 0)
+      (effects (font (size 1.27 1.27)) hide)
+    )
+    (property "MFG" "YAGEO" (at 67.31 118.11 0)
+      (effects (font (size 1.27 1.27)) hide)
+    )
+    (property "MFG_PN" "RC1206FR-071ML" (at 67.31 118.11 0)
+      (effects (font (size 1.27 1.27)) hide)
+    )
+    (property "Vendor1" "LCSC" (at 67.31 118.11 0)
+      (effects (font (size 1.27 1.27)) hide)
+    )
+    (property "Vendor1_PN" "C108083" (at 67.31 118.11 0)
+      (effects (font (size 1.27 1.27)) hide)
+    )
+    (property "Vendor1_URL" "https://www.lcsc.com/product-detail/Chip-Resistor-Surface-Mount_YAGEO-RC1206FR-071ML_C108083.html" (at 67.31 118.11 0)
       (effects (font (size 1.27 1.27)) hide)
     )
@@
       (effects (font (size 1.27 1.27)) hide)
     )
-    (property "Datasheet" "~" (at 134.62 85.09 0)
+    (property "Datasheet" "https://datasheet.lcsc.com/lcsc/2304140030_YAGEO-RC1206FR-075K1L_C163372.pdf" (at 134.62 85.09 0)
+      (effects (font (size 1.27 1.27)) hide)
+    )
+    (property "MFG" "YEGEO" (at 134.62 85.09 0)
+      (effects (font (size 1.27 1.27)) hide)
+    )
+    (property "MFG_PN" "RC1206FR-075K1L" (at 134.62 85.09 0)
+      (effects (font (size 1.27 1.27)) hide)
+    )
+    (property "Vendor1" "LCSC" (at 134.62 85.09 0)
+      (effects (font (size 1.27 1.27)) hide)
+    )
+    (property "Vendor1_PN" "C163372" (at 134.62 85.09 0)
+      (effects (font (size 1.27 1.27)) hide)
+    )
+    (property "Vendor1_URL" "https://www.lcsc.com/product-detail/Chip-Resistor-Surface-Mount_YAGEO-RC1206FR-075K1L_C163372.html" (at 134.62 85.09 0)
       (effects (font (size 1.27 1.27)) hide)
     )
@@
     )
   )
-  (symbol (lib_id "Device:R_Small_US") (at 142.24 81.28 0) (unit 1)
+  (symbol (lib_id "BadgePirates:R_5.1k_1206") (at 142.24 81.28 0) (unit 1)
     (in_bom yes) (on_board yes) (dnp no)
     (property "Reference" "R10" (at 143.9672 80.1116 0)
@@
       (effects (font (size 1.27 1.27)) hide)
     )
-    (property "Datasheet" "~" (at 142.24 81.28 0)
+    (property "Datasheet" "https://datasheet.lcsc.com/lcsc/2304140030_YAGEO-RC1206FR-075K1L_C163372.pdf" (at 142.24 81.28 0)
+      (effects (font (size 1.27 1.27)) hide)
+    )
+    (property "MFG" "YEGEO" (at 142.24 81.28 0)
+      (effects (font (size 1.27 1.27)) hide)
+    )
+    (property "MFG_PN" "RC1206FR-075K1L" (at 142.24 81.28 0)
+      (effects (font (size 1.27 1.27)) hide)
+    )
+    (property "Vendor1" "LCSC" (at 142.24 81.28 0)
+      (effects (font (size 1.27 1.27)) hide)
+    )
+    (property "Vendor1_PN" "C163372" (at 142.24 81.28 0)
+      (effects (font (size 1.27 1.27)) hide)
+    )
+    (property "Vendor1_URL" "https://www.lcsc.com/product-detail/Chip-Resistor-Surface-Mount_YAGEO-RC1206FR-075K1L_C163372.html" (at 142.24 81.28 0)
       (effects (font (size 1.27 1.27)) hide)
     )
@@
       (effects (font (size 1.27 1.27)) hide)
     )
-    (property "Datasheet" "~" (at 91.44 68.58 0)
+    (property "Datasheet" "https://datasheet.lcsc.com/lcsc/2206010200_UNI-ROYAL-Uniroyal-Elec-1206W4F0000T5E_C17888.pdf" (at 91.44 68.58 0)
+      (effects (font (size 1.27 1.27)) hide)
+    )
+    (property "MFG" "UNI-ROYAL(Uniroyal Elec) " (at 91.44 68.58 0)
+      (effects (font (size 1.27 1.27)) hide)
+    )
+    (property "MFG_PN" "1206W4F0000T5E" (at 91.44 68.58 0)
+      (effects (font (size 1.27 1.27)) hide)
+    )
+    (property "Vendor1" "LCSC" (at 91.44 68.58 0)
+      (effects (font (size 1.27 1.27)) hide)
+    )
+    (property "Vendor1_PN" "C17888" (at 91.44 68.58 0)
+      (effects (font (size 1.27 1.27)) hide)
+    )
+    (property "Vendor1_URL" "https://www.lcsc.com/product-detail/Chip-Resistor-Surface-Mount_UNI-ROYAL-Uniroyal-Elec-1206W4F0000T5E_C17888.html" (at 91.44 68.58 0)
       (effects (font (size 1.27 1.27)) hide)
     )
@@
     )
   )
-  (symbol (lib_id "Device:C_Small") (at 58.42 118.11 0) (unit 1)
+  (symbol (lib_id "BadgePirates:C_.1uf_0805") (at 58.42 118.11 0) (unit 1)
     (in_bom yes) (on_board yes) (dnp no)
     (property "Reference" "C8" (at 60.7568 116.9416 0)
@@
       (effects (font (size 1.27 1.27)) hide)
     )
-    (property "Datasheet" "~" (at 58.42 118.11 0)
+    (property "Datasheet" "https://datasheet.lcsc.com/lcsc/2304140030_TORCH-CT41G-0805-2X1-50V-0-1-F-K-N_C126469.pdf" (at 58.42 118.11 0)
+      (effects (font (size 1.27 1.27)) hide)
+    )
+    (property "MFG" "TORCH " (at 58.42 118.11 0)
+      (effects (font (size 1.27 1.27)) hide)
+    )
+    (property "MFG_PN" "CT41G-0805-2X1-50V-0.1μF-K(N)" (at 58.42 118.11 0)
+      (effects (font (size 1.27 1.27)) hide)
+    )
+    (property "Vendor1" "LCSC" (at 58.42 118.11 0)
+      (effects (font (size 1.27 1.27)) hide)
+    )
+    (property "Vendor1_PN" "C126469" (at 58.42 118.11 0)
+      (effects (font (size 1.27 1.27)) hide)
+    )
+    (property "Vendor1_URL" "https://www.lcsc.com/product-detail/Multilayer-Ceramic-Capacitors-MLCC-SMD-SMT_TORCH-CT41G-0805-2X1-50V-0-1-F-K-N_C126469.html" (at 58.42 118.11 0)
       (effects (font (size 1.27 1.27)) hide)
     )
@@
     )
     (property "Datasheet" "https://assets.nexperia.com/documents/data-sheet/PESD2USB3UV-T.pdf" (at 120.015 95.885 0)
+      (effects (font (size 1.27 1.27)) hide)
+    )
+    (property "MFG" "TECH PUBLIC" (at 116.84 99.06 0)
+      (effects (font (size 1.27 1.27)) hide)
+    )
+    (property "MFG_PN" "PESD2USB3UV-TR" (at 116.84 99.06 0)
+      (effects (font (size 1.27 1.27)) hide)
+    )
+    (property "Vendor1" "LCSC" (at 116.84 99.06 0)
+      (effects (font (size 1.27 1.27)) hide)
+    )
+    (property "Vendor_PN" "C7202955" (at 116.84 99.06 0)
+      (effects (font (size 1.27 1.27)) hide)
+    )
+    (property "Vendor1_URL" "https://www.lcsc.com/product-detail/span-style-background-color-ff0-ESD-span-Protection-Devices_TECH-PUBLIC-PESD2USB3UV-TR_C7202955.html" (at 116.84 99.06 0)
       (effects (font (size 1.27 1.27)) hide)
     )
@@
       (effects (font (size 1.27 1.27)) hide)
     )
+    (property "MFG" "Jing Extension of the Electronic Co." (at 74.93 88.9 0)
+      (effects (font (size 1.27 1.27)) hide)
+    )
+    (property "MFG_PN" "918-418K2023S40019" (at 74.93 88.9 0)
+      (effects (font (size 1.27 1.27)) hide)
+    )
+    (property "Vendor1" "LCSC" (at 74.93 88.9 0)
+      (effects (font (size 1.27 1.27)) hide)
+    )
+    (property "Vendor1_PN" "C709035" (at 74.93 88.9 0)
+      (effects (font (size 1.27 1.27)) hide)
+    )
+    (property "Vendor1_URL" "https://www.lcsc.com/product-detail/USB-Connectors_Jing-Extension-of-the-Electronic-Co-918-418K2023S40019_C709035.html" (at 74.93 88.9 0)
+      (effects (font (size 1.27 1.27)) hide)
+    )
