File: CAD/USB_Connections.kicad_sch (KiCad schematic)
At the start: 7 parts, among them J8 USB_C_Plug_USB2.0

Commit message: Updated part property names
Made part property names uniform
Parts:
- D19: Vendor1_PN (none) -> C7202955; Vendor_PN C7202955 -> (none)
Changed lines of the file:
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@@
       (effects (font (size 1.27 1.27)) hide)
     )
-    (property "Vendor_PN" "C7202955" (at 116.84 99.06 0)
+    (property "Vendor1_PN" "C7202955" (at 116.84 99.06 0)
       (effects (font (size 1.27 1.27)) hide)
     )

Commit message: fixing part numbers info on some parts
ESP, 340N, R330
Parts:
- D19: footprint Package_TO_SOT_SMD:SOT-23 -> BadgePirates:SOT-23
Changed lines of the file:
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@@
       (effects (font (size 1.27 1.27)) (justify left))
     )
-    (property "Footprint" "Package_TO_SOT_SMD:SOT-23" (at 122.555 100.33 0)
+    (property "Footprint" "BadgePirates:SOT-23" (at 122.555 100.33 0)
       (effects (font (size 1.27 1.27)) (justify left) hide)
     )
