File: CAD/Power.kicad_sch (KiCad schematic)
At the start: 11 parts, among them SW1 SW_SPDT, U1 LTC4054, U4 TLV1117LV33

Commit message: Schematic cleanup
Parts:
- added BT1: Battery, BadgePirates:Battery - 14500, symbol Device:Battery
- added F1: Fuse, BadgePirates:R_1206_3216Metric, symbol Device:Fuse
Connections:
- net BATTERY+: now also F1.1
- net GND: now also BT1.2 (-)
- new net: BT1.1 (+), F1.2
Other:
- moved on the sheet: BT1, C2, C6, C7, D10, F1, R2, R3, SW1, U1, U4

Commit message: Layout progress
Connections:
- net BATTERY2+: now reaches BT1.1 (+), F1.2
- net BATTERY2+: now also F1.1
- net BATTERY+ renamed BATTERY1+
- net BATTERY1+: no longer F1.1
Other:
- moved on the sheet: F1
Changed lines of the file:
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@@
   (junction (at 207.01 87.63) (diameter 0) (color 0 0 0 0)
   )
-  (junction (at 135.89 115.57) (diameter 0) (color 0 0 0 0)
-  )
   (junction (at 105.41 101.6) (diameter 0) (color 0 0 0 0)
   )
   (junction (at 177.8 87.63) (diameter 0) (color 0 0 0 0)
+  )
+  (junction (at 120.65 116.84) (diameter 0) (color 0 0 0 0)
   )
   (junction (at 135.89 90.17) (diameter 0) (color 0 0 0 0)
@@
     (stroke (width 0) (type default))
   )
-  (wire (pts (xy 120.65 115.57) (xy 120.65 118.11))
-    (stroke (width 0) (type default))
-  )
   (wire (pts (xy 196.85 130.81) (xy 208.28 130.81))
     (stroke (width 0) (type default))
@@
     (stroke (width 0) (type default))
   )
-  (wire (pts (xy 135.89 110.49) (xy 135.89 115.57))
+  (wire (pts (xy 120.65 116.84) (xy 125.73 116.84))
+    (stroke (width 0) (type default))
+  )
+  (wire (pts (xy 120.65 116.84) (xy 120.65 118.11))
     (stroke (width 0) (type default))
   )
@@
     (stroke (width 0) (type default))
   )
-  (wire (pts (xy 132.08 115.57) (xy 135.89 115.57))
+  (wire (pts (xy 133.35 116.84) (xy 135.89 116.84))
     (stroke (width 0) (type default))
   )
@@
     (stroke (width 0) (type default))
   )
+  (wire (pts (xy 135.89 110.49) (xy 120.65 110.49))
+    (stroke (width 0) (type default))
+  )
   (wire (pts (xy 161.29 116.84) (xy 166.37 116.84))
     (stroke (width 0) (type default))
@@
     (stroke (width 0) (type default))
   )
+  (wire (pts (xy 135.89 116.84) (xy 135.89 118.11))
+    (stroke (width 0) (type default))
+  )
   (wire (pts (xy 194.31 93.98) (xy 194.31 95.25))
     (stroke (width 0) (type default))
@@
     (stroke (width 0) (type default))
   )
+  (wire (pts (xy 120.65 110.49) (xy 120.65 116.84))
+    (stroke (width 0) (type default))
+  )
   (wire (pts (xy 161.29 83.82) (xy 161.29 87.63))
     (stroke (width 0) (type default))
@@
     (stroke (width 0) (type default))
   )
-  (wire (pts (xy 124.46 115.57) (xy 120.65 115.57))
-    (stroke (width 0) (type default))
-  )
   (wire (pts (xy 185.42 95.25) (xy 185.42 97.79))
-    (stroke (width 0) (type default))
-  )
-  (wire (pts (xy 135.89 115.57) (xy 135.89 118.11))
     (stroke (width 0) (type default))
   )
@@
     (effects (font (size 2.0066 2.0066)) (justify left bottom))
   )
-  (label "BATTERY+" (at 135.89 116.84 0) (fields_autoplaced)
+  (label "BATTERY2+" (at 120.65 110.49 0) (fields_autoplaced)
+    (effects (font (size 1.27 1.27)) (justify left bottom))
+  )
+  (label "BATTERY1+" (at 135.89 116.84 0) (fields_autoplaced)
     (effects (font (size 1.27 1.27)) (justify left bottom))
   )
@@
     )
   )
-  (symbol (lib_id "Device:Fuse") (at 128.27 115.57 270) (unit 1)
-    (in_bom yes) (on_board yes) (dnp no)
-    (property "Reference" "F1" (at 128.27 110.49 90)
-      (effects (font (size 1.27 1.27)))
-    )
-    (property "Value" "Fuse" (at 128.27 113.03 90)
-      (effects (font (size 1.27 1.27)))
-    )
-    (property "Footprint" "BadgePirates:R_1206_3216Metric" (at 128.27 113.792 90)
-      (effects (font (size 1.27 1.27)) hide)
-    )
-    (property "Datasheet" "~" (at 128.27 115.57 0)
-      (effects (font (size 1.27 1.27)) hide)
-    )
-    (property "OrderURL" "" (at 128.27 115.57 0)
-      (effects (font (size 1.27 1.27)) hide)
-    )
+  (symbol (lib_id "Device:Fuse") (at 129.54 116.84 270) (unit 1)
+    (in_bom yes) (on_board yes) (dnp no)
+    (property "Reference" "F1" (at 129.54 111.76 90)
+      (effects (font (size 1.27 1.27)))
+    )
+    (property "Value" "Fuse" (at 129.54 114.3 90)
+      (effects (font (size 1.27 1.27)))
+    )
+    (property "Footprint" "BadgePirates:R_1206_3216Metric" (at 129.54 115.062 90)
+      (effects (font (size 1.27 1.27)) hide)
+    )
+    (property "Datasheet" "~" (at 129.54 116.84 0)
+      (effects (font (size 1.27 1.27)) hide)
+    )
+    (property "OrderURL" "" (at 129.54 116.84 0)
+      (effects (font (size 1.27 1.27)) hide)
+    )

Commit message: Updated pins and moar
Parts:
- U4: MFG (none) -> Texas Instruments; MFG_PN (none) -> TLV1117LV33DCYR; MFN Texas Instruments -> (none); MFP TLV1117LV33DCYR -> (none)
Changed lines of the file:
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@@
       (effects (font (size 1.27 1.27)) hide)
     )
-    (property "MFN" "Texas Instruments" (at 185.42 87.63 0)
+    (property "MFG" "Texas Instruments" (at 185.42 87.63 0)
       (effects (font (size 1.27 1.27)) hide)
     )
-    (property "MFP" "TLV1117LV33DCYR" (at 185.42 87.63 0)
+    (property "MFG_PN" "TLV1117LV33DCYR" (at 185.42 87.63 0)
       (effects (font (size 1.27 1.27)) hide)
     )

Commit message: updates
Parts:
- BT1: MFG (none) -> Keystone Electronics; MFG_PN (none) -> 53; Vendor (none) -> DigiKey; Vendor1_PN (none) -> 36-53-ND; Vendor1_URL (none) -> https://www.digikey.com/en/products/detail/keystone-electro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
- BT1: symbol Device:Battery -> BadgePirates:Battery_Connector_14500_x2; MFG (none) -> Keystone Electronics; MFG_PN (none) -> 53; Vendor (none) -> DigiKey; Vendor1_PN (none) -> 36-53-ND; Vendor1_URL (none) -> https://www.digikey.com/en/products/detail/keystone-electro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
- C2: MFG (none) -> Samsung Electro-Mechanics; MFG_PN (none) -> CL21B105KBFNNNE; Vendor1 (none) -> LCSC; Vendor1_PN (none) -> C28323; Vendor1_URL (none) -> https://www.lcsc.com/product-detail/Multilayer-Ceramic-Capa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
- C6: symbol Device:C_Small -> BadgePirates:C_.1uf_0805; MFG (none) -> TORCH; MFG_PN (none) -> CT41G-0805-2X1-50V-0.1μF-K(N); Vendor1 (none) -> LCSC; Vendor1_PN (none) -> C126469; Vendor1_URL (none) -> https://www.lcsc.com/product-detail/Multilayer-Ceramic-Capa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
- C7: Package (none) -> CASE-B-3528; Vendor (none) -> LCSC; Vendor1_URL (none) -> https://www.lcsc.com/product-detail/Tantalum-Capacitors_Kyo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; Vendor_PN (none) -> C7195
- D10: MFG (none) -> Foshan NationStar Optoelectronics; MFG_PN (none) -> NCD1206B1; Vendor1 (none) -> LCSC; Vendor1_PN (none) -> C130717; Vendor1_URL (none) -> https://www.lcsc.com/product-detail/Light-Emitting-Diodes-s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
- F1: symbol Device:Fuse -> BadgePirates:Fuse; MFG (none) -> TLC Electronic; MFG_PN (none) -> TLC-NSMD200; Vendor1 (none) -> LCSC; Vendor1_PN (none) -> C261957; Vendor1_URL (none) -> https://www.lcsc.com/product-detail/Resettable-Fuses_TLC-El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
- F1: MFG (none) -> TLC Electronic; MFG_PN (none) -> TLC-NSMD200; Vendor1 (none) -> LCSC; Vendor1_PN (none) -> C261957; Vendor1_URL (none) -> https://www.lcsc.com/product-detail/Resettable-Fuses_TLC-El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
- R2: MFG (none) -> YAGEO; MFG_PN (none) -> RC1206FR-072KL; Vendor1 (none) -> LCSC; Vendor1_PN (none) -> C133543; Vendor1_URL (none) -> https://www.lcsc.com/product-detail/Chip-Resistor-Surface-M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
- SW1: value SW_SPDT -> On/Off; MFG (none) -> ALPSALPINE; MFG_PN (none) -> SSSS811101; Vendor1 (none) -> LCSC; Vendor1_PN (none) -> C109335; Vendor1_URL (none) -> https://www.lcsc.com/product-detail/Slide-Switches_ALPSALPI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
- U1: MFG (none) -> TPOWER; MFG_PN (none) -> TP4054ST25K; Vendor1 (none) -> LCSC; Vendor1_PN (none) -> TP4054ST25K; Vendor1_URL (none) -> https://www.lcsc.com/product-detail/Battery-Management-ICs_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
- U4: Vendor1 (none) -> LCSC; Vendor1_PN (none) -> C15578; Vendor1_URL (none) -> https://www.lcsc.com/product-detail/_Texas-Instruments-_C15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
