File: CAD/Power.kicad_sch (KiCad schematic)
At the start: 13 parts, among them SW1 On/Off, U1 LTC4054, U4 TLV1117LV33

Commit message: Updated part property names
Made part property names uniform
Parts:
- BT1: Vendor DigiKey -> (none); Vendor1 (none) -> DigiKey
- C7: MFG PN TAJB107M006RNJ -> (none); MFG_PN (none) -> TAJB107M006RNJ; Vendor LCSC -> (none); Vendor1 (none) -> LCSC; Vendor1_PN (none) -> C7195; Vendor_PN C7195 -> (none)
Changed lines of the file:
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@@
       (effects (font (size 1.27 1.27)) hide)
     )
-    (property "Vendor" "DigiKey" (at 135.89 123.19 0)
+    (property "Vendor1" "DigiKey" (at 135.89 123.19 0)
       (effects (font (size 1.27 1.27)) hide)
     )
@@
       (effects (font (size 1.27 1.27)) hide)
     )
-    (property "MFG PN" "TAJB107M006RNJ" (at 194.31 91.44 0)
-      (effects (font (size 1.27 1.27)) hide)
-    )
-    (property "Vendor" "LCSC" (at 194.31 91.44 0)
-      (effects (font (size 1.27 1.27)) hide)
-    )
-    (property "Vendor_PN" "C7195" (at 194.31 91.44 0)
+    (property "MFG_PN" "TAJB107M006RNJ" (at 194.31 91.44 0)
+      (effects (font (size 1.27 1.27)) hide)
+    )
+    (property "Vendor1" "LCSC" (at 194.31 91.44 0)
+      (effects (font (size 1.27 1.27)) hide)
+    )
+    (property "Vendor1_PN" "C7195" (at 194.31 91.44 0)
       (effects (font (size 1.27 1.27)) hide)
     )
@@
       (effects (font (size 1.27 1.27)) hide)
     )
-    (property "Vendor" "DigiKey" (at 120.65 123.19 0)
-      (effects (font (size 1.27 1.27)) hide)
-    )
+    (property "Vendor1" "DigiKey" (at 120.65 123.19 0)
+      (effects (font (size 1.27 1.27)) hide)
+    )

Commit message: fixing part numbers info on some parts
ESP, 340N, R330
Parts:
- R3: symbol Device:R_Small_US -> BadgePirates:R_330k_1206; MFG (none) -> YAGEO; MFG_PN (none) -> AC1206JR-07330KL; Vendor1 (none) -> LCSC; Vendor1_PN (none) -> C229929; Vendor1_URL (none) -> https://www.lcsc.com/product-detail/Chip-Resistor-Surface-M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
Changed lines of the file:
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@@
     )
   )
-  (symbol (lib_id "Device:R_Small_US") (at 83.82 82.55 0) (unit 1)
+  (symbol (lib_id "BadgePirates:R_330k_1206") (at 83.82 82.55 0) (unit 1)
     (in_bom yes) (on_board yes) (dnp no)
     (property "Reference" "R3" (at 85.5472 81.3816 0)
@@
       (effects (font (size 1.27 1.27)) hide)
     )
-    (property "Datasheet" "~" (at 83.82 82.55 0)
+    (property "Datasheet" "https://datasheet.lcsc.com/lcsc/2304140030_YAGEO-AC1206JR-07330KL_C229929.pdf" (at 83.82 82.55 0)
       (effects (font (size 1.27 1.27)) hide)
     )
@@
       (effects (font (size 1.27 1.27)) hide)
     )
+    (property "MFG" "YAGEO" (at 83.82 82.55 0)
+      (effects (font (size 1.27 1.27)) hide)
+    )
+    (property "MFG_PN" "AC1206JR-07330KL" (at 83.82 82.55 0)
+      (effects (font (size 1.27 1.27)) hide)
+    )
+    (property "Vendor1" "LCSC" (at 83.82 82.55 0)
+      (effects (font (size 1.27 1.27)) hide)
+    )
+    (property "Vendor1_PN" "C229929" (at 83.82 82.55 0)
+      (effects (font (size 1.27 1.27)) hide)
+    )
+    (property "Vendor1_URL" "https://www.lcsc.com/product-detail/Chip-Resistor-Surface-Mount_YAGEO-AC1206JR-07330KL_C229929.html" (at 83.82 82.55 0)
+      (effects (font (size 1.27 1.27)) hide)
+    )

Commit message: Update Power.kicad_sch
Parts:
- BT1: symbol Device:Battery -> BadgePirates:Battery_Connector_14500_x2
Changed lines of the file:
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@@
     )
   )
-  (symbol (lib_id "Device:Battery") (at 135.89 123.19 0) (unit 1)
+  (symbol (lib_id "BadgePirates:Battery_Connector_14500_x2") (at 135.89 123.19 0) (unit 1)
     (in_bom yes) (on_board yes) (dnp no) (fields_autoplaced)
-    (property "Reference" "BT1" (at 138.557 121.9005 0)
-      (effects (font (size 1.27 1.27)) (justify left))
-    )
-    (property "Value" "Battery" (at 138.557 124.6756 0)
+    (property "Reference" "BT1" (at 139.7 121.539 0)
+      (effects (font (size 1.27 1.27)) (justify left))
+    )
+    (property "Value" "Battery" (at 139.7 124.079 0)
       (effects (font (size 1.27 1.27)) (justify left))
     )
@@
       (effects (font (size 1.27 1.27)) hide)
     )
+    (pin "1")
+    (pin "2")
     (pin "1")
     (pin "2")
@@
     (pin "1")
     (pin "2")
+    (pin "1")
+    (pin "2")
