File: CAD/RotaryEncoders.kicad_sch (KiCad schematic)
At the start: 8 parts, among them SW9 RotaryEncoder_Switch

Commit message: Layout progress
Parts:
- SW9: footprint Rotary_Encoder:RotaryEncoder_Alps_EC11E_Vertical_H20mm_CircularMountingHoles -> Rotary_Encoder:RotaryEncoder_Alps_EC11E-Switch_Vertical_H20mm_CircularMountingHoles
Changed lines of the file:
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@@
       (effects (font (size 1.27 1.27)))
     )
-    (property "Footprint" "Rotary_Encoder:RotaryEncoder_Alps_EC11E_Vertical_H20mm_CircularMountingHoles" (at 78.74 58.166 0)
+    (property "Footprint" "Rotary_Encoder:RotaryEncoder_Alps_EC11E-Switch_Vertical_H20mm_CircularMountingHoles" (at 78.74 58.166 0)
       (effects (font (size 1.27 1.27)) hide)
     )
@@
       (effects (font (size 1.27 1.27)))
     )
-    (property "Footprint" "Rotary_Encoder:RotaryEncoder_Alps_EC11E_Vertical_H20mm_CircularMountingHoles" (at 77.47 115.316 0)
-      (effects (font (size 1.27 1.27)) hide)
-    )
+    (property "Footprint" "Rotary_Encoder:RotaryEncoder_Alps_EC11E-Switch_Vertical_H20mm_CircularMountingHoles" (at 77.47 115.316 0)
+      (effects (font (size 1.27 1.27)) hide)
+    )

Commit message: Updated pins and moar
Connections:
- net IO25 renamed IO20
Changed lines of the file:
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@@
     (effects (font (size 1.27 1.27)) (justify left bottom))
   )
-  (global_label "IO25" (shape input) (at 99.06 59.69 0) (fields_autoplaced)
+  (global_label "IO20" (shape input) (at 99.06 59.69 0) (fields_autoplaced)
     (effects (font (size 1.27 1.27)) (justify left))
-    (property "Intersheetrefs" "${INTERSHEET_REFS}" (at 105.6659 59.69 0)
+    (property "Intersheetrefs" "${INTERSHEET_REFS}" (at 105.7453 59.69 0)
       (effects (font (size 1.27 1.27)) (justify left) hide)
     )

Commit message: updates
Parts:
- R14, R15, R16: symbol Device:R_Small_US -> BadgePirates:R_10k_1206; MFG (none) -> YAGEO; MFG_PN (none) -> RC1206FR-0710KL; Vendor1 (none) -> LCSC; Vendor1_PN (none) -> C132649; Vendor1_URL (none) -> https://www.lcsc.com/product-detail/Chip-Resistor-Surface-M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
- SW9: MFG (none) -> ALPSALPINE; MFG_PN (none) -> EC11E1820402; Vendor1 (none) -> LCSC; Vendor1_PN (none) -> C361167; Vendor1_URL (none) -> https://www.lcsc.com/product-detail/Rotary-Encoders_ALPSALP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
- SW9: symbol Device:RotaryEncoder_Switch -> BadgePirates:RotaryEncoder_Switch; MFG (none) -> ALPSALPINE; MFG_PN (none) -> EC11E1820402; Vendor1 (none) -> LCSC; Vendor1_PN (none) -> C361167; Vendor1_URL (none) -> https://www.lcsc.com/product-detail/Rotary-Encoders_ALPSALP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
