File: CAD/Screens.kicad_sch (KiCad schematic)
At the start: 4 parts, among them J7 RoundDisplay_SPI, J9 RoundDisplay_SPI_v2

Commit message: updates
Parts:
- J7, J9: now not fitted
- R25: symbol Device:R_Small_US -> BadgePirates:R_4.7k_1206; MFG (none) -> YAGEO; MFG_PN (none) -> RT1206FRE074K7L; Vendor1 (none) -> LCSC; Vendor1_PN (none) -> C872804; Vendor1_URL (none) -> https://www.lcsc.com/product-detail/Chip-Resistor-Surface-M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
Changed lines of the file:
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@@
   )
   (symbol (lib_id "Connector:Conn_01x08_Pin") (at 180.34 77.47 0) (unit 1)
-    (in_bom yes) (on_board yes) (dnp no)
+    (in_bom yes) (on_board yes) (dnp yes)
     (property "Reference" "J9" (at 180.975 66.04 0)
       (effects (font (size 1.27 1.27)))
@@
   )
   (symbol (lib_id "Connector:Conn_01x07_Pin") (at 128.27 77.47 0) (unit 1)
-    (in_bom yes) (on_board yes) (dnp no)
+    (in_bom yes) (on_board yes) (dnp yes)
     (property "Reference" "J7" (at 128.905 66.04 0)
       (effects (font (size 1.27 1.27)))
@@
     )
   )
-  (symbol (lib_id "Device:R_Small_US") (at 153.67 72.39 0) (unit 1)
+  (symbol (lib_id "BadgePirates:R_4.7k_1206") (at 153.67 72.39 0) (unit 1)
     (in_bom yes) (on_board yes) (dnp no)
     (property "Reference" "R25" (at 155.3972 71.2216 0)
@@
       (effects (font (size 1.27 1.27)) hide)
     )
-    (property "Datasheet" "~" (at 153.67 72.39 0)
+    (property "Datasheet" "https://datasheet.lcsc.com/lcsc/2210181830_YAGEO-RT1206FRE074K7L_C872804.pdf" (at 153.67 72.39 0)
       (effects (font (size 1.27 1.27)) hide)
     )
     (property "OrderURL" "" (at 153.67 72.39 0)
+      (effects (font (size 1.27 1.27)) hide)
+    )
+    (property "MFG" "YAGEO" (at 153.67 72.39 0)
+      (effects (font (size 1.27 1.27)) hide)
+    )
+    (property "MFG_PN" "RT1206FRE074K7L" (at 153.67 72.39 0)
+      (effects (font (size 1.27 1.27)) hide)
+    )
+    (property "Vendor1" "LCSC" (at 153.67 72.39 0)
+      (effects (font (size 1.27 1.27)) hide)
+    )
+    (property "Vendor1_PN" "C872804" (at 153.67 72.39 0)
+      (effects (font (size 1.27 1.27)) hide)
+    )
+    (property "Vendor1_URL" "https://www.lcsc.com/product-detail/Chip-Resistor-Surface-Mount_YAGEO-RT1206FRE074K7L_C872804.html" (at 153.67 72.39 0)
       (effects (font (size 1.27 1.27)) hide)
     )
@@
     )
   )
-  (symbol (lib_id "Device:R_Small_US") (at 144.78 73.025 0) (unit 1)
+  (symbol (lib_id "BadgePirates:R_4.7k_1206") (at 144.78 73.025 0) (unit 1)
     (in_bom yes) (on_board yes) (dnp no)
     (property "Reference" "R25" (at 146.5072 71.8566 0)
@@
       (effects (font (size 1.27 1.27)) hide)
     )
-    (property "Datasheet" "~" (at 144.78 73.025 0)
+    (property "Datasheet" "https://datasheet.lcsc.com/lcsc/2210181830_YAGEO-RT1206FRE074K7L_C872804.pdf" (at 144.78 73.025 0)
       (effects (font (size 1.27 1.27)) hide)
     )
@@
       (effects (font (size 1.27 1.27)) hide)
     )
+    (property "MFG" "YAGEO" (at 144.78 73.025 0)
+      (effects (font (size 1.27 1.27)) hide)
+    )
+    (property "MFG_PN" "RT1206FRE074K7L" (at 144.78 73.025 0)
+      (effects (font (size 1.27 1.27)) hide)
+    )
+    (property "Vendor1" "LCSC" (at 144.78 73.025 0)
+      (effects (font (size 1.27 1.27)) hide)
+    )
+    (property "Vendor1_PN" "C872804" (at 144.78 73.025 0)
+      (effects (font (size 1.27 1.27)) hide)
+    )
+    (property "Vendor1_URL" "https://www.lcsc.com/product-detail/Chip-Resistor-Surface-Mount_YAGEO-RT1206FRE074K7L_C872804.html" (at 144.78 73.025 0)
+      (effects (font (size 1.27 1.27)) hide)
+    )
