File: CAD/Screens.kicad_sch (KiCad schematic)
At the start: 4 parts, among them J7 RoundDisplay_SPI, J9 RoundDisplay_SPI_v2

Commit message: adding art
Parts:
- removed J9: RoundDisplay_SPI_v2, Connector_PinSocket_2.54mm:PinSocket_1x08_P2.54mm_Vertical, symbol Connector:Conn_01x08_Pin
Changed lines of the file:
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@@
-    (stroke (width 0) (type default))
-  )
-  (wire (pts (xy 188.595 85.09) (xy 185.42 85.09))
-    (stroke (width 0) (type default))
-  )
-  (wire (pts (xy 188.595 77.47) (xy 185.42 77.47))
-    (stroke (width 0) (type default))
-  )
-  (wire (pts (xy 188.595 74.93) (xy 185.42 74.93))
     (stroke (width 0) (type default))
   )
@@
     (stroke (width 0) (type default))
   )
-  (wire (pts (xy 188.595 87.63) (xy 185.42 87.63))
-    (stroke (width 0) (type default))
-  )
-  (wire (pts (xy 188.595 82.55) (xy 185.42 82.55))
-    (stroke (width 0) (type default))
-  )
   (wire (pts (xy 158.115 80.01) (xy 153.67 80.01))
     (stroke (width 0) (type default))
@@
     (stroke (width 0) (type default))
   )
-  (wire (pts (xy 188.595 80.01) (xy 185.42 80.01))
-    (stroke (width 0) (type default))
-  )
   (global_label "IO02" (shape input) (at 133.35 72.39 0) (fields_autoplaced)
     (effects (font (size 1.27 1.27)) (justify left))
@@
     )
   )
-  (global_label "IO38" (shape input) (at 188.595 87.63 0) (fields_autoplaced)
-    (effects (font (size 1.27 1.27)) (justify left))
-    (property "Intersheetrefs" "${INTERSHEET_REFS}" (at 195.2009 87.63 0)
-      (effects (font (size 1.27 1.27)) (justify left) hide)
-    )
-  )
-  (global_label "IO21" (shape input) (at 188.595 80.01 0) (fields_autoplaced)
-    (effects (font (size 1.27 1.27)) (justify left))
-    (property "Intersheetrefs" "${INTERSHEET_REFS}" (at 195.2803 80.01 0)
-      (effects (font (size 1.27 1.27)) (justify left) hide)
-    )
-  )
-  (global_label "IO01" (shape input) (at 188.595 82.55 0) (fields_autoplaced)
-    (effects (font (size 1.27 1.27)) (justify left))
-    (property "Intersheetrefs" "${INTERSHEET_REFS}" (at 195.2009 82.55 0)
-      (effects (font (size 1.27 1.27)) (justify left) hide)
-    )
-  )
-  (global_label "IO09" (shape input) (at 188.595 74.93 0) (fields_autoplaced)
-    (effects (font (size 1.27 1.27)) (justify left))
-    (property "Intersheetrefs" "${INTERSHEET_REFS}" (at 195.2009 74.93 0)
-      (effects (font (size 1.27 1.27)) (justify left) hide)
-    )
-  )
   (global_label "IO08" (shape input) (at 158.115 77.47 0) (fields_autoplaced)
     (effects (font (size 1.27 1.27)) (justify left))
@@
     )
   )
-  (global_label "IO08" (shape input) (at 188.595 77.47 0) (fields_autoplaced)
-    (effects (font (size 1.27 1.27)) (justify left))
-    (property "Intersheetrefs" "${INTERSHEET_REFS}" (at 195.2009 77.47 0)
-      (effects (font (size 1.27 1.27)) (justify left) hide)
-    )
-  )
   (global_label "IO01" (shape input) (at 133.35 74.93 0) (fields_autoplaced)
     (effects (font (size 1.27 1.27)) (justify left))
@@
     )
   )
-  (global_label "IO02" (shape input) (at 188.595 85.09 0) (fields_autoplaced)
-    (effects (font (size 1.27 1.27)) (justify left))
-    (property "Intersheetrefs" "${INTERSHEET_REFS}" (at 195.2009 85.09 0)
-      (effects (font (size 1.27 1.27)) (justify left) hide)
-    )
-  )
-  (symbol (lib_name "VCC_1") (lib_id "power:VCC") (at 185.42 72.39 270) (unit 1)
-    (in_bom yes) (on_board yes) (dnp no)
-    (property "Reference" "#PWR068" (at 181.61 72.39 0)
-      (effects (font (size 1.27 1.27)) hide)
-    )
-    (property "Value" "VCC" (at 189.23 72.39 90)
-      (effects (font (size 1.27 1.27)) (justify left))
-    )
-    (property "Footprint" "" (at 185.42 72.39 0)
-      (effects (font (size 1.27 1.27)) hide)
-    )
-    (property "Datasheet" "" (at 185.42 72.39 0)
-      (effects (font (size 1.27 1.27)) hide)
-    )
-    (pin "1")
-    (instances
-      (project "ProjectNeoRogue"
-        (path "/76a22395-5d2d-4f66-8191-432f65fdc4ac/7bbc5ee4-a356-48de-a261-211ab35ec87b"
-          (reference "#PWR068") (unit 1)
-        )
-      )
-    )
-  )
   (symbol (lib_id "power:VCC") (at 144.78 67.31 0) (unit 1)
     (in_bom yes) (on_board yes) (dnp no)
@@
     )
   )
-  (symbol (lib_id "Connector:Conn_01x08_Pin") (at 180.34 77.47 0) (unit 1)
-    (in_bom no) (on_board yes) (dnp yes)
-    (property "Reference" "J9" (at 180.975 66.04 0)
-      (effects (font (size 1.27 1.27)))
-    )
-    (property "Value" "RoundDisplay_SPI_v2" (at 173.99 78.74 90)
-      (effects (font (size 1.27 1.27)))
-    )
-    (property "Footprint" "Connector_PinSocket_2.54mm:PinSocket_1x08_P2.54mm_Vertical" (at 180.34 77.47 0)
-      (effects (font (size 1.27 1.27)) hide)
-    )
-    (property "Datasheet" "~" (at 180.34 77.47 0)
+  (symbol (lib_id "Connector:Conn_01x07_Pin") (at 128.27 77.47 0) (unit 1)
+    (in_bom yes) (on_board yes) (dnp yes)
+    (property "Reference" "J7" (at 128.905 66.04 0)
+      (effects (font (size 1.27 1.27)))
+    )
+    (property "Value" "RoundDisplay_SPI" (at 124.46 77.47 90)
+      (effects (font (size 1.27 1.27)))
+    )
+    (property "Footprint" "Connector_PinSocket_2.54mm:PinSocket_1x07_P2.54mm_Vertical" (at 128.27 77.47 0)
+      (effects (font (size 1.27 1.27)) hide)
+    )
+    (property "Datasheet" "~" (at 128.27 77.47 0)
       (effects (font (size 1.27 1.27)) hide)
     )
@@
     (pin "6")
     (pin "7")
-    (pin "8")
-    (instances
-      (project "ProjectNeoRogue"
-        (path "/76a22395-5d2d-4f66-8191-432f65fdc4ac/7bbc5ee4-a356-48de-a261-211ab35ec87b"
-          (reference "J9") (unit 1)
-        )
-      )
-    )
-  )
-  (symbol (lib_id "Connector:Conn_01x07_Pin") (at 128.27 77.47 0) (unit 1)
-    (in_bom yes) (on_board yes) (dnp yes)
-    (property "Reference" "J7" (at 128.905 66.04 0)
-      (effects (font (size 1.27 1.27)))
-    )
-    (property "Value" "RoundDisplay_SPI" (at 124.46 77.47 90)
-      (effects (font (size 1.27 1.27)))
-    )
-    (property "Footprint" "Connector_PinSocket_2.54mm:PinSocket_1x07_P2.54mm_Vertical" (at 128.27 77.47 0)
-      (effects (font (size 1.27 1.27)) hide)
-    )
-    (property "Datasheet" "~" (at 128.27 77.47 0)
-      (effects (font (size 1.27 1.27)) hide)
-    )
-    (pin "1")
-    (pin "2")
-    (pin "3")
-    (pin "4")
-    (pin "5")
-    (pin "6")
-    (pin "7")
     (instances
       (project "ProjectNeoRogue"
@@
         )
       )
-    )
-  )
-  (symbol (lib_name "GND_1") (lib_id "power:GND") (at 185.42 69.85 90) (unit 1)
-    (in_bom yes) (on_board yes) (dnp no) (fields_autoplaced)
-    (property "Reference" "#PWR067" (at 191.77 69.85 0)
-      (effects (font (size 1.27 1.27)) hide)
-    )
-    (property "Value" "GND" (at 189.23 70.485 90)
-      (effects (font (size 1.27 1.27)) (justify right))
-    )
-    (property "Footprint" "" (at 185.42 69.85 0)
-      (effects (font (size 1.27 1.27)) hide)
-    )
-    (property "Datasheet" "" (at 185.42 69.85 0)
-      (effects (font (size 1.27 1.27)) hide)
-    )
-    (pin "1")
-    (instances
-      (project "ProjectNeoRogue"
-        (path "/76a22395-5d2d-4f66-8191-432f65fdc4ac/7bbc5ee4-a356-48de-a261-211ab35ec87b"
-          (reference "#PWR067") (unit 1)
-        )
-      )
