File: CAD/ProjectNeoRogue.kicad_pcb (KiCad board)
At the start: 4 copper layers, 95.5 x 113.7 mm, 87 parts, among them J1 5v GND, J10 Conn_01x01_Socket, J2 Micro_SD_Card, J3 JTAG, J4 UART, J5 Reset Jumper, J6 Boot Jumper, J7 RoundDisplay_SPI, J8 USB_C_Plug_USB2.0, J9 RoundDisplay_SPI_v2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

Commit message: adding artwork
Parts:
- added G***: LOGO, Footprints:F.Mask_Traces, F.Cu at (175.3, 101.3)
- added G***: LOGO, Footprints:F.Cu_LetterShadow, F.Cu at (237.7, 108.5)
- added G***: LOGO, Footprints:F.SilkS_Vee, F.Cu at (165.1, 124.1)
- added G***: LOGO, Footprints:F.SilkS_Main, F.Cu at (166.3, 100.0)
- added G***: LOGO, Footprints:F.Cu_Traces, F.Cu at (175.4, 101.3)
- added G***: LOGO, Footprints:F.Mask_LetterShadow, F.Cu at (237.7, 108.5)
- added G***: LOGO, Footprints:F.SilkS_Letters, F.Cu at (237.1, 107.7)
- added G***: LOGO, Footprints:F.Mask_Vee, F.Cu at (162.7, 81.5)

Commit message: adding art
Parts:
- removed C11: 100pF, Capacitor_SMD:C_0603_1608Metric_Pad1.08x0.95mm_HandSolder
- removed the G*** at (137.1, 113.8)
- removed J10: Conn_01x01_Socket, Connector_PinHeader_2.54mm:PinHeader_1x01_P2.54mm_Vertical
- removed J3: JTAG, Connector:Tag-Connect_TC2030-IDC-FP_2x03_P1.27mm_Vertical
- removed J5: Reset Jumper, BadgePirates:PinHeader_1x02_P2.54mm_Vertical
- removed J6: Boot Jumper, BadgePirates:PinHeader_1x02_P2.54mm_Vertical
- removed J9: RoundDisplay_SPI_v2, Connector_PinSocket_2.54mm:PinSocket_1x08_P2.54mm_Vertical
- removed R21: 75k, Resistor_SMD:R_0603_1608Metric_Pad0.98x0.95mm_HandSolder
- removed R22: 10K, BadgePirates:R_1206_3216Metric
- removed R24: 22k, BadgePirates:R_1206_3216Metric
- added REF**: 5.5mm, BadgePirates:Hole_5.5mm, F.Cu at (214.3, 103.3)
- moved R15 128.2 mm to (125.3, 57.6), turned to -90 degrees
- moved R16 114.3 mm to (147.7, 53.0)
- moved SW9 114.0 mm to (128.0, 51.1)
- moved R14 92.8 mm to (125.3, 49.8), turned to 90 degrees
- moved D8 63.5 mm to (203.1, 149.2)
- moved D7 61.4 mm to (203.3, 143.0)
- moved D6 59.0 mm to (203.5, 136.6)
- moved X1 58.7 mm to (210.6, 53.6), turned to -90 degrees
- moved R9 56.4 mm to (192.8, 149.3)
- moved J7 53.0 mm to (168.0, 128.3), turned to 90 degrees
- moved SW3 48.8 mm to (179.7, 49.5)
- moved SW2 40.9 mm to (171.3, 49.4)
- moved R23 32.0 mm to (176.2, 92.0)
- moved R27 30.5 mm to (181.7, 92.0), turned to 0 degrees
- moved J1 26.8 mm to (152.8, 156.8), turned to 90 degrees
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Routing:
- net IO05: track 166.2 -> 22.8 mm, vias 10 -> 2
- net IO20: track 135.5 -> 19.1 mm, vias 4 -> 2
- net IO04: track 142.8 -> 29.0 mm, vias 7 -> 2
- net Net-(D7-A): track 11.5 -> 61.5 mm, vias 0 -> 2
- net IO01: track 107.7 -> 155.6 mm, vias 4 -> 3
- net Net-(JP3-A): track 3.94 -> 50.5 mm
- net Net-(D6-A): track 14.5 -> 59.7 mm, vias 0 -> 2
- net IO38: track 41.8 -> 0.00 mm
- net IO15: track 94.3 -> 132.6 mm, vias 2 -> 4
- net IO18: track 80.6 -> 50.7 mm
- net VBUS: track 88.8 -> 61.5 mm
- net Net-(JP2-B): track 6.14 -> 31.6 mm
- net TCK: track 24.2 -> 0.00 mm
- net TMS: track 21.5 -> 0.00 mm
- net Net-(D11-DOUT): track 5.70 -> 22.7 mm
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- added copper zone on F.Cu, net (none)
Other:
- outline, holes or cut-outs redrawn

Commit message: cleanup and screen shots of 3d View
Parts:
- added G***: LOGO, BadgePirates_Logos:BadgePiratesURL_B.SLK, F.Cu at (174.2, 73.3)
- added G***: BP Logo, BadgePirates_Logos:BPSkull_Distressed_B.SILK, F.Cu at (183.2, 73.5)
- added REF**: 5.5mm, BadgePirates:Hole_5.5mm, F.Cu at (214.4, 49.5)
- moved REF** 52.3 mm to (214.7, 155.7)
- moved X1 13.9 mm to (211.9, 67.4)
- moved G*** 12.5 mm to (201.4, 158.1)
- moved D9 12.4 mm to (201.4, 155.5)
- moved R1 7.83 mm to (207.1, 155.5), turned to 180 degrees
Routing:
- net Net-(JP2-B): track 31.6 -> 48.4 mm
- net Net-(JP3-A): track 50.5 -> 66.2 mm
- net IO07: track 177.5 -> 164.0 mm, vias 3 -> 4
- net IO06: track 191.2 -> 178.3 mm
- net GND: track 24.2 -> 26.1 mm
- net Net-(D9-A): track 4.10 -> 2.96 mm

Commit message: Gerbers and BOM
Parts:
- added Fid-1: Fiducial_1mm_Mask2mm, Fiducial:Fiducial_1mm_Mask2mm, B.Cu at (146.9, 48.8)
- added Fid-2: Fiducial_1mm_Mask2mm, Fiducial:Fiducial_1mm_Mask2mm, B.Cu at (215.5, 102.1)
- added Fid-3: Fiducial_1mm_Mask2mm, Fiducial:Fiducial_1mm_Mask2mm, B.Cu at (124.5, 158.0)
- added Fid-4: Fiducial_0.5mm_Mask1mm, Fiducial:Fiducial_0.5mm_Mask1mm, F.Cu at (176.6, 88.7)
- added Fid-5: Fiducial_0.5mm_Mask1mm, Fiducial:Fiducial_0.5mm_Mask1mm, F.Cu at (193.4, 109.0)
- added Fid-6: Fiducial_0.5mm_Mask1mm, Fiducial:Fiducial_0.5mm_Mask1mm, F.Cu at (162.9, 112.9)
- added G***: Rixon, BadgePirates_Logos:rixon_B.Cu, F.Cu at (150.6, 148.1)
- D19: value PESD2USB3UV-TR -> PESD
- J8: value USB_C_Plug_USB2.0 -> USB_C
- moved REF** 5.85 mm to (152.8, 134.5)
- moved G*** 3.63 mm to (144.8, 128.7)
- moved R20 1.42 mm to (198.8, 129.3)
- moved U5 1.10 mm to (205.0, 131.1)
- moved D19 1.04 mm to (170.7, 146.6), turned to 90 degrees
- moved R11 0.86 mm to (166.8, 146.9)
- moved R10 0.32 mm to (174.9, 147.0)
Routing:
- net IO01: track 155.6 -> 122.4 mm
- net IO02: track 101.2 -> 82.3 mm, vias 3 -> 1
- net IO08: track 91.6 -> 86.1 mm
- net GND: track 26.1 -> 22.5 mm, vias 38 -> 36
- net IO10: track 58.6 -> 55.0 mm, vias 4 -> 2
- net IO45: track 64.4 -> 61.2 mm
- net IO18: track 50.7 -> 48.1 mm, vias 3 -> 1
- net D-: track 15.8 -> 18.4 mm, vias 2 -> 0
- net IO17: track 125.6 -> 123.1 mm
- net IO04: track 29.0 -> 26.9 mm
- net Net-(J8-VBUS-PadA4): track 17.8 -> 16.1 mm
- net IO06: track 178.3 -> 176.7 mm
- net +BATT: track 44.0 -> 45.3 mm
- net IO15: track 132.6 -> 131.3 mm
- net IO46: track 21.1 -> 20.1 mm
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Other:
- board text added: "Thank You"

Commit message: working on code
Parts:
- removed the G*** at (237.7, 108.5) (x2)
- removed the G*** at (237.1, 107.7)
- added G***: LOGO, Footprints:F.Cu_NewTextShadow, F.Cu at (237.7, 104.6)
- added G***: LOGO, Footprints:F.Mask_NewTextShadow, F.Cu at (245.0, 104.4)
- added G***: LOGO, Footprints:F.SilkS_NewLettersTop, F.Cu at (237.2, 107.7)
Other:
- board text added: "TGFzdCBCYWRnZSwgdHkgQlA="
- board text removed: "Thank You"
