File: CAD/CactusCon12.kicad_sch (KiCad schematic)
At the start: 27 parts, among them J1 5v GND, J2 Micro_SD_Card, J4 UART, SW2 Boot, SW3 Reset, U2 ESP32-S3-WROOM-1, U3 CH340N, X1 sao_v169bis

Commit message: Cleaning up
Other:
- title: Project_NeoRogue -> CactusCon12
